File: variable voltage battery charger 1/variable voltage battery charger 1.kicad_sch (KiCad schematic)
At the start: 0 parts

Commit message: Add files via upload
Parts:
- added C1: 330uF, Capacitor_THT:CP_Radial_D8.0mm_P5.00mm, symbol Device:C_Polarized_US
- added D1, D2, D3, D4: 1N4001, Diode_THT:D_DO-41_SOD81_P10.16mm_Horizontal, symbol Diode:1N4001
- added GREEN1: LED, LED_THT:LED_D3.0mm_Clear, symbol Device:LED
- added J1, J2: Conn_01x02_Pin, Connector_PinSocket_2.54mm:PinSocket_1x02_P2.54mm_Vertical, symbol Connector:Conn_01x02_Pin
- added K1: JQC-3FF-005-1Z, Relay_THT:Relay_SPDT_Hongfa_JQC-3FF_0XX-1Z, symbol Relay:JQC-3FF-005-1Z
- added R1: 220 ohm, Resistor_THT:R_Axial_DIN0207_L6.3mm_D2.5mm_P7.62mm_Horizontal, symbol Device:R
- added R2: 1K, Resistor_THT:R_Axial_DIN0207_L6.3mm_D2.5mm_P7.62mm_Horizontal, symbol Device:R
- added RED1: LED, LED_THT:LED_D3.0mm, symbol Device:LED
- added RV1, RV2: 10K, Potentiometer_THT:Potentiometer_Bourns_3296W_Vertical, symbol Device:R_Potentiometer_Trim
- added U1: LM317_TO-220, Package_TO_SOT_THT:TO-220-3_Vertical, symbol Regulator_Linear:LM317_TO-220
Connections:
- new net: D3.2 (A), D4.1 (K), J1.2 (Pin_2)
- new net: C1.2, D2.2 (A), D4.2 (A), J2.1 (Pin_1), R2.2, RV1.1, RV2.1
- new net: K1.A2, RV2.2
- new net: D1.2 (A), D2.1 (K), J1.1 (Pin_1)
- new net: R1.2, RV1.2, U1.1 (ADJ)
- new net: GREEN1.1 (K), R2.1, RED1.1 (K)
- new net: C1.1, D1.1 (K), D3.1 (K), U1.3 (VI)
- new net: K1.11, K1.A1, R1.1, U1.2 (VO)
- new net: GREEN1.2 (A), K1.14
- new net: J2.2 (Pin_2), K1.12, RED1.2 (A)
